File: pcb/ConnDIN41612.kicad_sch (KiCad schematic)
At the start: 40 parts, among them IC1 SN65HVD75DR, J1 DIN41612_02x32_AC, T1 H1102NL, U3 USBLC6-2SC6, U4 USBLC6-2SC6, U5 USBLC6-2SC6

Commit message: Little cleaning
Parts:
- T1: footprint SOIC127P940X597-16N -> SamacSys_Parts:SOIC127P940X597-16N
Changed lines of the file:
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@@
 			)
 		)
-		(property "Footprint" "SOIC127P940X597-16N"
+		(property "Footprint" "SamacSys_Parts:SOIC127P940X597-16N"
 			(at 115.57 234.62 0)
 			(effects
