File: pcb/EthernetPHY.kicad_sch (KiCad schematic)
At the start: 24 parts, among them U1 W5500, Y2 3225-25M-SR

Commit message: Edited Resistor array to be included in bom
Parts:
- RN1, RN2, RN3: now in the parts list
Changed lines of the file:
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@@
 		(unit 1)
 		(exclude_from_sim no)
-		(in_bom no)
+		(in_bom yes)
 		(on_board yes)
 		(dnp no)
@@
 		(unit 1)
 		(exclude_from_sim no)
-		(in_bom no)
+		(in_bom yes)
 		(on_board yes)
 		(dnp no)
@@
 		(unit 1)
 		(exclude_from_sim no)
-		(in_bom no)
-		(on_board yes)
-		(dnp no)
+		(in_bom yes)
+		(on_board yes)
+		(dnp no)
