File: pcb/EthernetPHY.kicad_sch (KiCad schematic)
At the start: 24 parts, among them U1 W5500, Y2 3225-25M-SR

Commit message: Modification based on prototype
Parts:
- Y2: symbol Device:Crystal_GND23 -> Device:Crystal_GND24
Connections:
- net GND: now also Y2.4; no longer Y2.3
- net XO-: now also Y2.3; no longer Y2.4
Changed lines of the file:
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@@
 	)
 	(symbol
-		(lib_id "Device:Crystal_GND23")
+		(lib_id "Device:Crystal_GND24")
 		(at 86.36 114.3 0)
 		(unit 1)
@@
 			)
 		)
-		(property "Description" "Four pin crystal, GND on pins 2 and 3"
+		(property "Description" "Four pin crystal, GND on pins 2 and 4"
 			(at 86.36 114.3 0)
 			(effects
