File: pcb/MCU.kicad_sch (KiCad schematic)
At the start: 19 parts, among them J2 TC2030, J3 Conn_01x02_Pin, U2 STM32G431CBTx, U6 FM24C64B, Y1 3225-25M-SR

Commit message: Modification based on prototype
Parts:
- Y1: symbol Device:Crystal_GND23 -> Device:Crystal_GND24
Connections:
- net GND: now also Y1.4; no longer Y1.3
- net XTAL-: now also Y1.3; no longer Y1.4
Changed lines of the file:
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@@
 	)
 	(symbol
-		(lib_id "Device:Crystal_GND23")
+		(lib_id "Device:Crystal_GND24")
 		(at 81.28 95.25 0)
 		(unit 1)
@@
 			)
 		)
-		(property "Description" "Four pin crystal, GND on pins 2 and 3"
+		(property "Description" "Four pin crystal, GND on pins 2 and 4"
 			(at 81.28 95.25 0)
 			(effects
