File: pcb/RDE_board.kicad_pcb (KiCad board)
At the start: 2 copper layers, 160 x 100 mm, 383 parts, among them IC1 SN65HVD75DR, IC101 STPIC6C595TTR, IC102 STPIC6C595TTR, IC103 STPIC6C595TTR, IC104 STPIC6C595TTR, IC105 STPIC6C595TTR, IC106 STPIC6C595TTR, J1 DIN41612_02x32_AC, J2 TC2030, J3 Conn_01x02_Pin, J4 7772, J5 7772, J6 7772, J7 7772, K1 TQ2-5V, K10 TQ2-5V, K11 TQ2-5V, K12 TQ2-5V, K13 TQ2-5V, K14 TQ2-5V, K15 TQ2-5V, K16 TQ2-5V, K17 TQ2-5V, K18 TQ2-5V, K19 TQ2-5V, K2 TQ2-5V, K20 TQ2-5V, K21 TQ2-5V, K22 TQ2-5V, K23 TQ2-5V, K24 TQ2-5V, K25 TQ2-5V, K26 TQ2-5V, K27 TQ2-5V, K28 TQ2-5V, K29 TQ2-5V, K3 TQ2-5V, K30 TQ2-5V, K31 TQ2-5V, K32 TQ2-5V, K33 TQ2-5V, K34 TQ2-5V, K35 TQ2-5V, K36 TQ2-5V, K37 TQ2-5V, K38 TQ2-5V, K39 TQ2-5V, K4 TQ2-5V, K5 TQ2-5V, K6 TQ2-5V, K7 TQ2-5V, K8 TQ2-5V, K9 TQ2-5V, Q1 BSS138, T1 H1102NL, U1 W5500, U2 STM32G431CBTx, U3 USBLC6-2SC6, U4 USBLC6-2SC6, U5 USBLC6-2SC6, U6 FM24C64B, Y1 3225-25M-SR, Y2 3225-25M-SR

Commit message: Modification based on prototype
Parts:
- added R92: 1, Resistor_SMD:R_0603_1608Metric_Pad0.98x0.95mm_HandSolder, F.Cu at (1.68, 0.76)
- added R93: 2, Resistor_SMD:R_0603_1608Metric_Pad0.98x0.95mm_HandSolder, F.Cu at (1.68, 3.27)
- added R94: 2, Resistor_SMD:R_0603_1608Metric_Pad0.98x0.95mm_HandSolder, F.Cu at (1.68, 5.78)
- added R95: 2, Resistor_SMD:R_0603_1608Metric_Pad0.98x0.95mm_HandSolder, F.Cu at (1.68, 8.29)
- added R96: 2, Resistor_SMD:R_0603_1608Metric_Pad0.98x0.95mm_HandSolder, F.Cu at (1.68, 10.8)
Connections:
- C1 pad 1: +5V -> +3.3V
- C2 pad 1: +5V -> +3.3V
- U4 pad 5: +5V -> +3.3V
- U5 pad 5: +5V -> +3.3V
- Y1 pad 3: GND -> /MCU/XTAL-
- Y1 pad 4: /MCU/XTAL- -> GND
- Y2 pad 3: GND -> /EthernetPHY/XO-
- Y2 pad 4: /EthernetPHY/XO- -> GND
Routing:
- net +5V: track 136.4 -> 113.8 mm, vias 5 -> 3
- net +3.3V: track 170.2 -> 189.3 mm, vias 19 -> 21
